File: HPA2.kicad_sch (KiCad schematic)
At the start: 120 parts, among them J1 Input, J2 Conn_01x01_Male, J3 Power, J4 Output, J5 Mute, K1 EA2-12NJ, Q1 BC560C, Q10 BC560C, Q11 BC560C, Q12 BC549C, Q13 BC549C, Q14 KSC1845, Q15 BC549C, Q16 BC560C, Q17 KSA992, Q18 BC560C, Q19 BC550C, Q2 BC559C, Q20 BC560C, Q21 BC550C, Q22 TTA004B, Q23 TTA004B, Q24 TTC004B, Q25 TTC004B, Q26 KSC2690AY, Q27 KSA1220AY, Q3 BC549C, Q4 BC549C, Q5 BC549C, Q6 BC559C, Q7 BC549C, Q8 BC560C, Q9 BC560C, U1 2N5564, U2 LT1761-BYP, U3 LT1964-BYP, U4 ADA4627-1

Commit message: On the schematic: - Aligned schematic to grid. - Changed all default library transistor symbols to generic Q_PNP/Q_NPN symbols. - Updated other out-of-date default library symbols - Added GND_PWR flags to fix ERC errors.
Parts:
- C18, C19: symbol HPA2-rescue:CP1-Device -> Device:C_Polarized_US
- J1, J4, J5: symbol HPA2-rescue:Conn_01x02_Male-Connector -> Connector:Conn_01x02_Pin
- J2: symbol HPA2-rescue:Conn_01x01_Male-Connector -> Connector:Conn_01x01_Pin
- J3: symbol HPA2-rescue:Conn_01x03_Male-Connector -> Connector:Conn_01x03_Pin
- Q1, Q10, Q11, Q16, Q18, Q2, Q20, Q6, Q8, Q9: symbol Transistor_BJT:BC560 -> Transistor_BJT:Q_PNP_CBE
- Q12, Q13, Q15, Q19, Q21, Q3, Q4, Q5, Q7: symbol Transistor_BJT:BC550 -> Transistor_BJT:Q_NPN_CBE
- Q14, Q26: symbol Device:Q_NPN_ECB -> Transistor_BJT:Q_NPN_ECB
- Q17, Q27: symbol Device:Q_PNP_ECB -> Transistor_BJT:Q_PNP_ECB
- Q22, Q23: symbol Transistor_BJT:BD140 -> Transistor_BJT:Q_PNP_ECB
- Q24, Q25: symbol Transistor_BJT:BD139 -> Transistor_BJT:Q_NPN_ECB
Connections:
- net at C3.2, D10.1 (K), D9.2 (A)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: now also D11.2 (A), Q11.2 (B), Q17.3 (B), Q8.1 (C), Q9.1 (C)
Other:
- moved on the sheet: C1, C10, C11, C12, C13, C14, C15, C17, C18, C19, C2, C20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

Commit message: - Created project-local symbol library - Copied custom 2N5564, CRD, and ADA4627-1 symbols to the library - Deleted HPA2-rescue library
Parts:
- D1, D6: symbol HPA2-rescue:CRD-HP_Miscellaneous -> HPA2_symbols:CRD
- U1: symbol HPA2-rescue:2N5564-HP-Transistor_FET -> HPA2_symbols:2N5564
- U4: symbol HPA2-rescue:ADA4627-1-HP_Op_Amps -> HPA2_symbols:ADA4627-1
Changed lines of the file:
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@@
 	)
 	(symbol
-		(lib_id "HPA2-rescue:2N5564-HP-Transistor_FET")
+		(lib_id "HPA2_symbols:2N5564")
 		(at 139.7 172.72 0)
 		(mirror y)
@@
 	)
 	(symbol
-		(lib_id "HPA2-rescue:CRD-HP_Miscellaneous")
+		(lib_id "HPA2_symbols:CRD")
 		(at 132.08 209.55 90)
 		(unit 1)
@@
 	)
 	(symbol
-		(lib_id "HPA2-rescue:CRD-HP_Miscellaneous")
+		(lib_id "HPA2_symbols:CRD")
 		(at 109.22 113.03 90)
 		(unit 1)
@@
 	)
 	(symbol
-		(lib_id "HPA2-rescue:ADA4627-1-HP_Op_Amps")
+		(lib_id "HPA2_symbols:ADA4627-1")
 		(at 302.26 312.42 180)
 		(unit 1)

Commit message: Updated schematic to be consistent with PCB footprint changes.
Parts:
- C10, C9: footprint Capacitor_SMD:C_0805_2012Metric_Pad1.15x1.40mm_HandSolder -> Capacitor_SMD:C_0805_2012Metric_Pad1.18x1.45mm_HandSolder
- D1, D6: footprint HP_Footprints:Semitec-CRD-SMD -> HPA2-footprints:Semitec-CRD-SMD
- D10, D11, D12, D13, D14, D15, D16, D17, D9: footprint Diode_THT:D_DO-35_SOD27_P7.62mm_Horizontal -> HPA2-footprints:D_DO-35_SOD27_P7.62mm_Horizontal
- D2, D3, D4: footprint Diode_THT:D_DO-34_SOD68_P7.62mm_Horizontal -> HPA2-footprints:D_DO-34_SOD68_P7.62mm_Horizontal
- J1, J4: footprint HP_Footprints:2-pad-wire-connector-small -> HPA2-footprints:2-pad-wire-connector-small
- J2: footprint HP_Footprints:1-pad-wire-connector-22-ga -> HPA2-footprints:1-pad-wire-connector-22-ga
- J3: footprint HP_Footprints:3-pad-wire-connector-22-ga -> HPA2-footprints:3-pad-wire-connector-22-ga
- J5: footprint HP_Footprints:2-pad-wire-connector-22-ga -> HPA2-footprints:2-pad-wire-connector-22-ga
- L1: footprint HP_Footprints:HPA-Output-Coil -> HPA2-footprints:HPA-Output-Coil
- Q22, Q23, Q24, Q25, Q26, Q27: footprint Package_TO_SOT_THT:TO-126-3_Vertical -> HPA2-footprints:TO-126-3_Vertical
- R26, R27, R28, R29, R34, R35: footprint Resistor_SMD:R_0805_2012Metric_Pad1.15x1.40mm_HandSolder -> HPA2-footprints:R_0805_2012Metric_Pad1.15x1.40mm_HandSolder
- U1: footprint HP_Footprints:TO-71-6 -> HPA2-footprints:TO-71-6
- U2, U3: footprint Package_TO_SOT_SMD:TSOT-23-5 -> HPA2-footprints:TSOT-23-5
Connections:
- net at C3.2, D10.1 (K), D9.2 (A)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: no longer D11.2 (A), Q11.2 (B), Q17.3 (B), Q8.1 (C), Q9.1 (C)
- new net: D11.2 (A), Q11.2 (B), Q17.3 (B), Q8.1 (C), Q9.1 (C)
Changed lines of the file:
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@@
 	)
 	(junction
-		(at 175.26 132.08)
-		(diameter 0)
-		(color 0 0 0 0)
-	)
-	(junction
 		(at 139.7 246.38)
 		(diameter 0)
@@
 	(wire
 		(pts
-			(xy 175.26 132.08) (xy 162.56 132.08)
+			(xy 162.56 132.08) (xy 190.5 132.08)
 		)
 		(stroke
@@
 	(wire
 		(pts
-			(xy 190.5 132.08) (xy 175.26 132.08)
-		)
-		(stroke
-			(width 0)
-			(type default)
-		)
-	)
-	(wire
-		(pts
 			(xy 279.4 317.5) (xy 274.32 317.5)
 		)
@@
 			)
 		)
-		(property "Footprint" "HP_Footprints:TO-71-6"
+		(property "Footprint" "HPA2-footprints:TO-71-6"
 			(at 139.7 182.88 0)
 			(effects
@@
 			)
 		)
-		(property "Footprint" "HP_Footprints:Semitec-CRD-SMD"
+		(property "Footprint" "HPA2-footprints:Semitec-CRD-SMD"
 			(at 136.525 209.55 0)
 			(effects
@@
 			)
 		)
-		(property "Footprint" "Package_TO_SOT_THT:TO-126-3_Vertical"
+		(property "Footprint" "HPA2-footprints:TO-126-3_Vertical"
 			(at 378.46 130.175 0)
 			(effects
@@
 			)
 		)
-		(property "Footprint" "Package_TO_SOT_THT:TO-126-3_Vertical"
+		(property "Footprint" "HPA2-footprints:TO-126-3_Vertical"
 			(at 378.46 182.245 0)
 			(effects
@@
 			)
 		)
-		(property "Footprint" "Package_TO_SOT_THT:TO-126-3_Vertical"
+		(property "Footprint" "HPA2-footprints:TO-126-3_Vertical"
 			(at 378.46 215.265 0)
 			(effects
@@
 			)
 		)
-		(property "Footprint" "HP_Footprints:3-pad-wire-connector-22-ga"
+		(property "Footprint" "HPA2-footprints:3-pad-wire-connector-22-ga"
 			(at 444.5 124.46 0)
 			(effects
@@
 			)
 		)
-		(property "Footprint" "HP_Footprints:Semitec-CRD-SMD"
+		(property "Footprint" "HPA2-footprints:Semitec-CRD-SMD"
 			(at 113.665 113.03 0)
 			(effects
@@
 			)
 		)
-		(property "Footprint" "HP_Footprints:2-pad-wire-connector-22-ga"
+		(property "Footprint" "HPA2-footprints:2-pad-wire-connector-22-ga"
 			(at 485.14 205.74 0)
 			(effects
@@
 			)
 		)
-		(property "Footprint" "Resistor_SMD:R_0805_2012Metric_Pad1.15x1.40mm_HandSolder"
+		(property "Footprint" "HPA2-footprints:R_0805_2012Metric_Pad1.15x1.40mm_HandSolder"
 			(at 303.022 227.33 90)
 			(effects
@@
 			)
 		)
-		(property "Footprint" "Resistor_SMD:R_0805_2012Metric_Pad1.15x1.40mm_HandSolder"
+		(property "Footprint" "HPA2-footprints:R_0805_2012Metric_Pad1.15x1.40mm_HandSolder"
 			(at 303.022 240.03 90)
 			(effects
@@
 			)
 		)
-		(property "Footprint" "Diode_THT:D_DO-35_SOD27_P7.62mm_Horizontal"
+		(property "Footprint" "HPA2-footprints:D_DO-35_SOD27_P7.62mm_Horizontal"
 			(at 461.01 210.185 0)
 			(effects
@@
 			)
 		)
-		(property "Footprint" "Diode_THT:D_DO-35_SOD27_P7.62mm_Horizontal"
+		(property "Footprint" "HPA2-footprints:D_DO-35_SOD27_P7.62mm_Horizontal"
 			(at 140.97 117.475 0)
 			(effects
@@
 			)
 		)
-		(property "Footprint" "Capacitor_SMD:C_0805_2012Metric_Pad1.15x1.40mm_HandSolder"
+		(property "Footprint" "Capacitor_SMD:C_0805_2012Metric_Pad1.18x1.45mm_HandSolder"
 			(at 302.26 252.4252 0)
 			(effects
@@
 			)
 		)
-		(property "Footprint" "Package_TO_SOT_THT:TO-126-3_Vertical"
+		(property "Footprint" "HPA2-footprints:TO-126-3_Vertical"
 			(at 403.86 142.24 0)
 			(effects
@@
 			)
 		)
-		(property "Footprint" "Package_TO_SOT_THT:TO-126-3_Vertical"
+		(property "Footprint" "HPA2-footprints:TO-126-3_Vertical"
 			(at 403.86 200.66 0)
 			(effects
@@
 			)
 		)
-		(property "Footprint" "Diode_THT:D_DO-34_SOD68_P7.62mm_Horizontal"
+		(property "Footprint" "HPA2-footprints:D_DO-34_SOD68_P7.62mm_Horizontal"
 			(at 109.22 153.67 0)
 			(effects
@@
 			)
 		)
-		(property "Footprint" "Diode_THT:D_DO-34_SOD68_P7.62mm_Horizontal"
+		(property "Footprint" "HPA2-footprints:D_DO-34_SOD68_P7.62mm_Horizontal"
 			(at 279.4 146.05 0)
 			(effects
@@
 			)
 		)
-		(property "Footprint" "Diode_THT:D_DO-34_SOD68_P7.62mm_Horizontal"
+		(property "Footprint" "HPA2-footprints:D_DO-34_SOD68_P7.62mm_Horizontal"
 			(at 279.4 199.39 0)
 			(effects
@@
 			)
 		)
-		(property "Footprint" "Resistor_SMD:R_0805_2012Metric_Pad1.15x1.40mm_HandSolder"
+		(property "Footprint" "HPA2-footprints:R_0805_2012Metric_Pad1.15x1.40mm_HandSolder"
 			(at 321.31 313.182 90)
 			(effects
@@
 			)
 		)
-		(property "Footprint" "Resistor_SMD:R_0805_2012Metric_Pad1.15x1.40mm_HandSolder"
+		(property "Footprint" "HPA2-footprints:R_0805_2012Metric_Pad1.15x1.40mm_HandSolder"
 			(at 321.31 290.322 90)
 			(effects
@@
 			)
 		)
-		(property "Footprint" "Package_TO_SOT_SMD:TSOT-23-5"
+		(property "Footprint" "HPA2-footprints:TSOT-23-5"
 			(at 320.04 80.01 0)
 			(effects
@@
 			)
 		)
-		(property "Footprint" "Package_TO_SOT_SMD:TSOT-23-5"
+		(property "Footprint" "HPA2-footprints:TSOT-23-5"
 			(at 322.58 251.46 0)
 			(effects
@@
 			)
 		)
-		(property "Footprint" "Resistor_SMD:R_0805_2012Metric_Pad1.15x1.40mm_HandSolder"
+		(property "Footprint" "HPA2-footprints:R_0805_2012Metric_Pad1.15x1.40mm_HandSolder"
 			(at 303.022 95.25 90)
 			(effects
@@
 			)
 		)
-		(property "Footprint" "Resistor_SMD:R_0805_2012Metric_Pad1.15x1.40mm_HandSolder"
+		(property "Footprint" "HPA2-footprints:R_0805_2012Metric_Pad1.15x1.40mm_HandSolder"
 			(at 303.022 107.95 90)
 			(effects
@@
 			)
 		)
-		(property "Footprint" "Package_TO_SOT_THT:TO-126-3_Vertical"
+		(property "Footprint" "HPA2-footprints:TO-126-3_Vertical"
 			(at 378.46 163.195 0)
 			(effects
@@
 			)
 		)
-		(property "Footprint" "HP_Footprints:2-pad-wire-connector-small"
+		(property "Footprint" "HPA2-footprints:2-pad-wire-connector-small"
 			(at 485.14 175.26 0)
 			(effects
@@
 			)
 		)
-		(property "Footprint" "Capacitor_SMD:C_0805_2012Metric_Pad1.15x1.40mm_HandSolder"
+		(property "Footprint" "Capacitor_SMD:C_0805_2012Metric_Pad1.18x1.45mm_HandSolder"
 			(at 299.72 82.2452 0)
 			(effects
@@
 			)
 		)
-		(property "Footprint" "HP_Footprints:2-pad-wire-connector-small"
+		(property "Footprint" "HPA2-footprints:2-pad-wire-connector-small"
 			(at 60.96 172.72 0)
 			(effects
@@
 			)
 		)
-		(property "Footprint" "Diode_THT:D_DO-35_SOD27_P7.62mm_Horizontal"
+		(property "Footprint" "HPA2-footprints:D_DO-35_SOD27_P7.62mm_Horizontal"
 			(at 380.365 153.67 0)
 			(effects
@@
 			)
 		)
-		(property "Footprint" "Diode_THT:D_DO-35_SOD27_P7.62mm_Horizontal"
+		(property "Footprint" "HPA2-footprints:D_DO-35_SOD27_P7.62mm_Horizontal"
 			(at 380.365 191.77 0)
 			(effects
@@
 			)
 		)
-		(property "Footprint" "HP_Footprints:HPA-Output-Coil"
+		(property "Footprint" "HPA2-footprints:HPA-Output-Coil"
 			(at 433.07 172.72 0)
 			(effects
@@
 			)
 		)
-		(property "Footprint" "Diode_THT:D_DO-35_SOD27_P7.62mm_Horizontal"
+		(property "Footprint" "HPA2-footprints:D_DO-35_SOD27_P7.62mm_Horizontal"
 			(at 140.97 121.285 0)
 			(effects
@@
 			)
 		)
-		(property "Footprint" "HP_Footprints:1-pad-wire-connector-22-ga"
+		(property "Footprint" "HPA2-footprints:1-pad-wire-connector-22-ga"
 			(at 302.26 193.04 0)
 			(effects
@@
 			)
 		)
-		(property "Footprint" "Diode_THT:D_DO-35_SOD27_P7.62mm_Horizontal"
+		(property "Footprint" "HPA2-footprints:D_DO-35_SOD27_P7.62mm_Horizontal"
 			(at 260.35 210.185 0)
 			(effects
@@
 			)
 		)
-		(property "Footprint" "Diode_THT:D_DO-35_SOD27_P7.62mm_Horizontal"
+		(property "Footprint" "HPA2-footprints:D_DO-35_SOD27_P7.62mm_Horizontal"
 			(at 260.35 205.105 0)
 			(effects
@@
 			)
 		)
-		(property "Footprint" "Diode_THT:D_DO-35_SOD27_P7.62mm_Horizontal"
+		(property "Footprint" "HPA2-footprints:D_DO-35_SOD27_P7.62mm_Horizontal"
 			(at 260.35 144.145 0)
 			(effects
@@
 			)
 		)
-		(property "Footprint" "Diode_THT:D_DO-35_SOD27_P7.62mm_Horizontal"
+		(property "Footprint" "HPA2-footprints:D_DO-35_SOD27_P7.62mm_Horizontal"
 			(at 260.35 151.765 0)
 			(effects
